File: Hardware/pedal/pedal.kicad_pcb (KiCad board)
At the start: 4 copper layers, 90 x 70 mm, 134 parts, among them J101 USB_C_Receptacle_USB2.0_16P, J102 Barrel_Jack_Switch, J103 AudioJack3_SwitchTR, J201 AudioJack4, J202 AudioJack4, J301 AudioJack3_SwitchTR, J302 AudioJack3_SwitchTR, SW101 SW_SPST, SW102 SW_SPST, SW103 RotaryEncoder_Switch_MP, U101 USBLC6-2P6, U102 TPS62153, U103 TLV76733DRVx, U201 SN74AHCT1G125DCKR, U202 TLP2310, U301 OPA2365AIDR, U302 TLV76733DRVx, U303 TAC5242, U401 APS6404L-3SQRx-ZR, U402 RP2354A, Y401 ABM8-272-T3

Commit message: Start re-doing the 'pedal' part without any actual audio processing
The 'minimal' board is what I think is the right way to go, and works
very well.  Being able to use WebMIDI over BLE just means that it's a
lot more convenient to use from a phone or a computer.

But as an actual *pedal* that minimal board isn't great.  It
intentionally has no actual physical controls, and since it's USB-C only
it doesn't work well on a traditional pedal board anyway.

But the plan was always to make things a bit more modular.  This is the
beginnings of that.  The non-minimal 'pedal' design has stomp switches
and hardware MIDI connectors and an expression pedal jack, and those all
worked fine.  It also has the traditional guitar pedal 9V DC jack.

So this just removes the actual audio side of it and only leaves that
cheap and useful rp2354 as the control piece and USB controller (it
never grew BLE support).  But now the main use of USB is as a USB
_host_, and as a way to power the minimal board.  It still presents as a
USB device for programming purposes, but that's now _purely_ for
programming.

[ Side note: the USB CC lines still claim it's acting as a USB device -
  exactly for that programming case. The minimal pedal doesn't care. All
  it wants is USB data lines and VBUS, so that "USB host" side is a bit
  dodgy from a USB standard side, but I can't find it in myself to
  really care. This isn't designed as some kind of generic USB host,
  it's designed explicitly as just a host for the minimal pedal design ]

So the usage scenario is that you connect your 9V guitar power to this
pedal, and use it as a pedal: it has the stomp switch and all controls
on it.  Then you snake the USB-C cable to the minimal box, which is
where you connect the audio to, and where all audio processing takes
place.

The pedal still has a TRS 6.35mm jack and two TRS 3.5mm jacks, but they
are purely for the remove switch (or expression pedal) and the Type-A
TRS MIDI connections.  No actual audio anywhere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
Parts:
- removed C301, C302, C303, C305, C310, C318, C321, C322: 2.2uF, Capacitor_SMD:C_0603_1608Metric
- removed C304, C309, C311, C312: 2.2nF, Capacitor_SMD:C_0402_1005Metric
- removed C306, C323, C326, C327, C404: 0.1uF, Capacitor_SMD:C_0402_1005Metric
- removed C307, C308: 150pF, Capacitor_SMD:C_0402_1005Metric
- removed C313, C314, C315, C316: 4.7uF, Capacitor_SMD:C_0805_2012Metric
- removed C317: 22uF, Capacitor_SMD:C_1210_3225Metric
- removed C319, C320, C324, C325: 10uF, Capacitor_SMD:C_0603_1608Metric
- removed D101: 1N5819WS, Diode_SMD:D_SOD-323
- removed D105, D107: BAT54SW, Package_TO_SOT_SMD:SOT-323_SC-70
- removed J301, J302: AudioJack3_SwitchTR, Mylib:NRJ6HM-1-PRE
- removed L301: 2.2uH, Mylib:L_0806
- removed R301, R302, R304, R305, R306, R310: 1MEG, Resistor_SMD:R_0402_1005Metric
- removed R303, R309: 1k, Resistor_SMD:R_0402_1005Metric
- removed R307, R308, R311, R312: 100R, Resistor_SMD:R_0402_1005Metric
- removed R313: 1R, Resistor_SMD:R_0402_1005Metric
- removed R401: 2.2kΩ, Resistor_SMD:R_0402_1005Metric
- removed U301: OPA2365AIDR, Package_SO:SOIC-8_3.9x4.9mm_P1.27mm
- removed U302: TLV76733DRVx, Package_SON:WSON-6-1EP_2x2mm_P0.65mm_EP1x1.6mm
- removed U303: TAC5242, Mylib:TAC5242
- removed U401: APS6404L-3SQRx-ZR, Package_SON:Winbond_USON-8-1EP_3x2mm_P0.5mm_EP0.2x1.6mm
- added R108: 100k, Resistor_SMD:R_0402_1005Metric, F.Cu at (60.4, 85.0)
- added U104: USBLC6-2P6, Package_TO_SOT_SMD:SOT-666, F.Cu at (130.6, 104.8)
- moved C108 38.9 mm to (132.2, 102.3), turned to -90 degrees
- moved R106 36.4 mm to (131.2, 102.3), turned to -90 degrees
- moved C105 35.0 mm to (128.9, 102.3)
- moved R104 34.6 mm to (129.9, 102.3), turned to -90 degrees
Connections:
- C107 pad 1: +5V -> VBUS
- C201 pad 2: +5V -> VBUS
- C203 pad 2: +5V -> VBUS
- C204 pad 2: +5V -> VBUS
- C205 pad 2: +5V -> VBUS
- C206 pad 2: +5V -> VBUS
- C207 pad 2: +5V -> VBUS
- D104 pad 1: +5V -> VBUS
- D202 pad 2: +5V -> VBUS
- D203 pad 2: +5V -> VBUS
- D204 pad 2: +5V -> VBUS
- D205 pad 2: +5V -> VBUS
- D206 pad 2: +5V -> VBUS
- J103 pad R: /EXP_R -> Net-(J103-PadR)
- J103 pad T: /EXP_T -> Net-(J103-PadT)
- R103 pad 2: +5V -> VBUS
- R104 pad 2: /EXP_T -> Net-(R104-Pad2)
- R106 pad 2: /EXP_R -> Net-(R106-Pad2)
- R202 pad 1: +5V -> VBUS
- U102 pad 8: GND -> /DEF
- U103 pad 6: +5V -> VBUS
- U201 pad 5: +5V -> VBUS
- U402 pad 32: /TAC5242/I2S.DIN -> /RP2354/GPIO20
- U402 pad 33: /TAC5242/I2S.DOUT -> /RP2354/GPIO21
- U402 pad 34: /TAC5242/I2S.FSYNC -> /RP2354/GPIO22
- U402 pad 35: /TAC5242/I2S.BCLK -> /RP2354/GPIO23
- U402 pad 55: /RP2354/SD3 -> unconnected-(U402-QSPI_SD3-Pad55)
- U402 pad 56: /RP2354/SCLK -> unconnected-(U402-QSPI_SCLK-Pad56)
- U402 pad 57: /RP2354/SD0 -> unconnected-(U402-QSPI_SD0-Pad57)
- U402 pad 58: /RP2354/SD2 -> unconnected-(U402-QSPI_SD2-Pad58)
- U402 pad 59: /RP2354/SD1 -> unconnected-(U402-QSPI_SD1-Pad59)
Routing:
- net +5V: track 191.2 -> 0.00 mm, vias 8 -> 0
- net VBUS: track 25.0 -> 151.9 mm, vias 4 -> 11
- net +3.3VA: track 53.4 -> 0.00 mm, vias 6 -> 0
- net /TAC5242/I2S.DIN: track 48.4 -> 0.00 mm
- net /TAC5242/I2S.DOUT: track 47.4 -> 0.00 mm
- net /TAC5242/I2S.FSYNC: track 46.5 -> 0.00 mm
- net /TAC5242/I2S.BCLK: track 45.5 -> 0.00 mm
- net /EXP_R: track 44.0 -> 0.00 mm, vias 1 -> 0
- net /EXP_T: track 37.0 -> 0.00 mm, vias 1 -> 0
- net +3V3: track 140.2 -> 118.2 mm, vias 17 -> 14
- net /TAC5242/OUT^{RIGHT}: track 17.0 -> 0.00 mm
- net /TAC5242/OUT^{LEFT}: track 16.7 -> 0.00 mm
- net GND: track 23.4 -> 11.9 mm, vias 109 -> 40
- net /RP2354/ADC1: track 15.8 -> 4.36 mm
- net Net-(C301-Pad2): track 10.3 -> 0.00 mm
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