File: Hardware/pedal/rp2354.kicad_sch (KiCad schematic)
At the start: 33 parts, among them U401 APS6404L-3SQRx-ZR, U402 RP2354A, Y401 ABM8-272-T3

Commit message: Start re-doing the 'pedal' part without any actual audio processing
The 'minimal' board is what I think is the right way to go, and works
very well.  Being able to use WebMIDI over BLE just means that it's a
lot more convenient to use from a phone or a computer.

But as an actual *pedal* that minimal board isn't great.  It
intentionally has no actual physical controls, and since it's USB-C only
it doesn't work well on a traditional pedal board anyway.

But the plan was always to make things a bit more modular.  This is the
beginnings of that.  The non-minimal 'pedal' design has stomp switches
and hardware MIDI connectors and an expression pedal jack, and those all
worked fine.  It also has the traditional guitar pedal 9V DC jack.

So this just removes the actual audio side of it and only leaves that
cheap and useful rp2354 as the control piece and USB controller (it
never grew BLE support).  But now the main use of USB is as a USB
_host_, and as a way to power the minimal board.  It still presents as a
USB device for programming purposes, but that's now _purely_ for
programming.

[ Side note: the USB CC lines still claim it's acting as a USB device -
  exactly for that programming case. The minimal pedal doesn't care. All
  it wants is USB data lines and VBUS, so that "USB host" side is a bit
  dodgy from a USB standard side, but I can't find it in myself to
  really care. This isn't designed as some kind of generic USB host,
  it's designed explicitly as just a host for the minimal pedal design ]

So the usage scenario is that you connect your 9V guitar power to this
pedal, and use it as a pedal: it has the stomp switch and all controls
on it.  Then you snake the USB-C cable to the minimal box, which is
where you connect the audio to, and where all audio processing takes
place.

The pedal still has a TRS 6.35mm jack and two TRS 3.5mm jacks, but they
are purely for the remove switch (or expression pedal) and the Type-A
TRS MIDI connections.  No actual audio anywhere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
Parts:
- removed C404: 0.1uF, Capacitor_SMD:C_0402_1005Metric, symbol Device:C
- removed R401: 2.2kΩ, Resistor_SMD:R_0402_1005Metric, symbol Device:R
- removed U401: APS6404L-3SQRx-ZR, Package_SON:Winbond_USON-8-1EP_3x2mm_P0.5mm_EP0.2x1.6mm, symbol Memory_RAM:APS6404L-3SQRx-ZR
Connections:
- net SCLK: no longer names the net of U402.56 (QSPI_SCLK)
- net SD0: no longer names the net of U402.57 (QSPI_SD0)
- net SD1: no longer names the net of U402.59 (QSPI_SD1)
- net SD2: no longer names the net of U402.58 (QSPI_SD2)
- net SD3: no longer names the net of U402.55 (QSPI_SD3)
- no-connect marks 0 -> 5
